Commit message: test to commit external folder

File: src/turtlebot3/turtlebot3_description/urdf/turtlebot3_waffle.gazebo.xacro (robot description, xacro)
@@ -1,5 +1,5 @@
 <?xml version="1.0"?>
 <robot name="turtlebot3_waffle_sim" xmlns:xacro="http://ros.org/wiki/xacro">
-  <xacro:arg name="laser_visual"  default="false"/>
+  <xacro:arg name="laser_visual"  default="true"/>
   <xacro:arg name="camera_visual" default="false"/>
   <xacro:arg name="imu_visual"    default="false"/>
@@ -105,6 +105,6 @@
     <material>Gazebo/FlatBlack</material>
     <sensor type="ray" name="lds_lfcd_sensor">
-      <pose>0 0 0 0 0 0</pose>
-      <visualize>$(arg laser_visual)</visualize>
+      <pose>0 0 10 0 0 0</pose>
+      <visualize>true</visualize>
       <update_rate>5</update_rate>
       <ray>

File: src/turtlebot3/turtlebot3_description/urdf/turtlebot3_waffle.urdf.xacro (robot description, xacro)
@@ -22,5 +22,5 @@
     </visual>
     <collision>
-      <origin xyz="-0.064 0 0.047" rpy="0 0 0"/>
+      <origin xyz="-0.064 0 0" rpy="0 0 0"/>
       <geometry>
         <box size="0.266 0.266 0.094"/>
